File: EEprom_Logger_V1.brd (EAGLE design)
At the start: 45.7 x 45.7 mm, 18 parts, among them IC1 TC1016, IC2 PIC18F13K22SOP, IC3 MIC94090, IC4 24LCS21ASN, Q2 Si2333CDS-T1-GE3, Y1 32kHz

Commit message: Add files via upload
Parts:
- removed IC4: 24LCS21ASN, microchip:SO-08
- removed VBATT: Vbatt, SparkFun-Connectors:JST-2-PTH
- added IC5: 24LC16BSN, microchip:SO-08
- added R2, R3: 4.7k, SparkFun-Resistors:1206
Connections:
- removed net VCC: IC4.8
- new net SCL: IC2.11, IC5.6, R2.1
- new net SDA: IC2.13, IC5.5, R3.1
- net GND: now also IC5.1, IC5.2, IC5.3, IC5.4, IC5.7; no longer IC4.4, VBATT.2
- net SWITCHED_VCC: now also IC5.8, R2.2, R3.2
- net VIN: no longer VBATT.1
Changed lines of the file:
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@@
 <?xml version="1.0" encoding="utf-8"?>
 <!DOCTYPE eagle SYSTEM "eagle.dtd">
-<eagle version="9.4.2">
+<eagle version="9.1.0">
 <drawing>
 <settings>
@@
 <attribute name="PROD_ID" value="TRANS-08285" x="4.826" y="24.384" size="1.778" layer="27" display="off"/>
 </element>
-<element name="VBATT" library="SparkFun-Connectors" package="JST-2-PTH" value="Vbatt" x="6.35" y="12.7" smashed="yes" rot="R90">
-<attribute name="SKU" value="PRT-09914" x="6.35" y="12.7" size="1.778" layer="27" rot="R90" display="off"/>
-</element>
 <element name="JP7" library="SparkFun-Connectors" package="JST-2-PTH" value="Vsolar" x="6.096" y="31.242" smashed="yes" rot="R90">
 <attribute name="NAME" x="0.826" y="29.972" size="0.4064" layer="25" rot="R90"/>
@@
 <attribute name="NAME" x="1.651" y="16.764" size="0.8128" layer="25" rot="R90"/>
 </element>
-<element name="IC4" library="microchip" library_urn="urn:adsk.eagle:library:294" package="SO-08" package3d_urn="urn:adsk.eagle:package:20804/2" value="24LCS21ASN" x="-6.35" y="0" smashed="yes">
-<attribute name="MF" value="MICROCHIP" x="-6.35" y="0" size="1.778" layer="27" display="off"/>
-<attribute name="MPN" value="24LCS21A/SN" x="-6.35" y="0" size="1.778" layer="27" display="off"/>
-<attribute name="NAME" x="-9.017" y="-1.905" size="1.27" layer="25" rot="R90"/>
-<attribute name="OC_FARNELL" value="1847803" x="-6.35" y="0" size="1.778" layer="27" display="off"/>
-<attribute name="OC_NEWARK" value="92C7025" x="-6.35" y="0" size="1.778" layer="27" display="off"/>
-<attribute name="VALUE" x="-2.413" y="-1.905" size="1.27" layer="27" rot="R90"/>
-</element>
+<element name="IC5" library="microchip" library_urn="urn:adsk.eagle:library:294" package="SO-08" package3d_urn="urn:adsk.eagle:package:20804/2" value="24LC16BSN" x="39.37" y="10.922">
+<attribute name="MF" value="MICROCHIP" x="39.37" y="10.922" size="1.778" layer="27" display="off"/>
+<attribute name="MPN" value="24LC16B/SN" x="39.37" y="10.922" size="1.778" layer="27" display="off"/>
+<attribute name="OC_FARNELL" value="9757945" x="39.37" y="10.922" size="1.778" layer="27" display="off"/>
+<attribute name="OC_NEWARK" value="12C2012" x="39.37" y="10.922" size="1.778" layer="27" display="off"/>
+</element>
+<element name="R2" library="SparkFun-Resistors" package="1206" value="4.7k" x="31.496" y="5.842" rot="R180"/>
+<element name="R3" library="SparkFun-Resistors" package="1206" value="4.7k" x="31.496" y="2.794" rot="R180"/>
 </elements>
 <signals>
@@
 <contactref element="IC1" pad="2"/>
 <contactref element="Q2" pad="1"/>
-<contactref element="VBATT" pad="2"/>
 <polygon width="0.4064" layer="1" isolate="0.4064">
 <vertex x="0" y="43.18"/>
@@
 <wire x1="8.636" y1="17.526" x2="8.128" y2="17.526" width="0.4064" layer="1"/>
 <wire x1="8.128" y1="17.526" x2="8.128" y2="17.018" width="0.4064" layer="1"/>
-<contactref element="IC4" pad="4"/>
-<wire x1="37.846" y1="19.558" x2="34.224" y2="12.446" width="0" layer="19" extent="1-1"/>
-<wire x1="-4.445" y1="-2.6" x2="6.35" y2="13.7" width="0" layer="19" extent="1-1"/>
+<contactref element="IC5" pad="4"/>
+<contactref element="IC5" pad="1"/>
+<contactref element="IC5" pad="2"/>
+<contactref element="IC5" pad="3"/>
+<contactref element="IC5" pad="7"/>
+<wire x1="32.226" y1="33.147" x2="41.497" y2="33.147" width="0" layer="19" extent="1-1"/>
+<wire x1="22.701" y1="33.147" x2="32.226" y2="33.147" width="0" layer="19" extent="1-1"/>
+<wire x1="18.288" y1="25.574" x2="22.701" y2="33.147" width="0" layer="19" extent="1-1"/>
+<wire x1="14.732" y1="28.448" x2="18.288" y2="25.574" width="0" layer="19" extent="1-1"/>
+<wire x1="14.732" y1="21.336" x2="18.288" y2="25.574" width="0" layer="19" extent="1-1"/>
+<wire x1="11.618" y1="23.384" x2="14.732" y2="21.336" width="0" layer="19" extent="1-1"/>
+<wire x1="8.636" y1="19.177" x2="11.618" y2="23.384" width="0" layer="19" extent="1-1"/>
+<wire x1="2.794" y1="20.45" x2="7.65" y2="19.177" width="0" layer="19" extent="1-1"/>
+<wire x1="3.876" y1="23.384" x2="2.794" y2="20.45" width="0" layer="19" extent="1-1"/>
+<wire x1="6.096" y1="32.242" x2="3.876" y2="23.384" width="0" layer="19" extent="1-1"/>
+<wire x1="37.846" y1="19.558" x2="41.497" y2="33.147" width="0" layer="19" extent="1-1"/>
+<wire x1="38.735" y1="13.522" x2="37.846" y2="19.558" width="0" layer="19" extent="1-1"/>
+<wire x1="34.29" y1="12.3825" x2="38.735" y2="13.522" width="0" layer="19" extent="1-1"/>
+<wire x1="37.465" y1="8.322" x2="34.29" y2="12.3825" width="0" layer="19" extent="1-1"/>
+<wire x1="38.735" y1="8.322" x2="37.465" y2="8.322" width="0" layer="19" extent="1-1"/>
+<wire x1="40.005" y1="8.322" x2="38.735" y2="8.322" width="0" layer="19" extent="1-1"/>
+<wire x1="41.275" y1="8.322" x2="40.005" y2="8.322" width="0" layer="19" extent="1-1"/>
+<wire x1="21.59" y1="7.236" x2="34.224" y2="12.446" width="0" layer="19" extent="1-1"/>
+<wire x1="18.542" y1="7.236" x2="21.59" y2="7.236" width="0" layer="19" extent="1-1"/>
 </signal>
 <signal name="PGD">
@@
 <contactref element="IC1" pad="1"/>
 <contactref element="Q2" pad="2"/>
-<contactref element="VBATT" pad="1"/>
 <wire x1="6.0325" y1="20.32" x2="6.0325" y2="23.1775" width="0.254" layer="1"/>
 <wire x1="7.62" y1="20.32" x2="6.6675" y2="20.32" width="0.254" layer="1"/>
@@
 <wire x1="1.27" y1="19.05" x2="1.27" y2="16.8275" width="0.254" layer="1"/>
 <wire x1="6.6675" y1="19.05" x2="1.27" y2="19.05" width="0.254" layer="1"/>
-<wire x1="6.35" y1="11.7475" x2="6.35" y2="11.7" width="0.254" layer="1"/>
 </signal>
 <signal name="ENABLE">
@@
 <wire x1="28.2575" y1="33.02" x2="28.2575" y2="23.495" width="0.254" layer="16"/>
 <wire x1="28.2575" y1="33.02" x2="28.226" y2="33.147" width="0.254" layer="16"/>
+<contactref element="IC5" pad="8"/>
+<contactref element="R3" pad="2"/>
+<contactref element="R2" pad="2"/>
 <wire x1="34.224" y1="11.796" x2="28.2575" y2="23.495" width="0" layer="19" extent="1-16"/>
-</signal>
-<signal name="VCC">
-<contactref element="IC4" pad="8"/>
+<wire x1="37.465" y1="13.522" x2="18.701" y2="33.147" width="0" layer="19" extent="1-1"/>
+<wire x1="30.096" y1="5.842" x2="37.465" y2="13.522" width="0" layer="19" extent="1-1"/>
+<wire x1="30.096" y1="2.794" x2="30.096" y2="5.842" width="0" layer="19" extent="1-1"/>
+</signal>
+<signal name="SDA">
+<contactref element="IC5" pad="5"/>
+<contactref element="R3" pad="1"/>
+<contactref element="IC2" pad="13"/>
+<wire x1="41.275" y1="13.522" x2="27.178" y2="25.574" width="0" layer="19" extent="1-1"/>
+<wire x1="32.896" y1="2.794" x2="41.275" y2="13.522" width="0" layer="19" extent="1-1"/>
+</signal>
+<signal name="SCL">
+<contactref element="IC5" pad="6"/>
+<contactref element="R2" pad="1"/>
+<contactref element="IC2" pad="11"/>
+<wire x1="40.005" y1="13.522" x2="29.718" y2="25.574" width="0" layer="19" extent="1-1"/>
+<wire x1="32.896" y1="5.842" x2="40.005" y2="13.522" width="0" layer="19" extent="1-1"/>
 </signal>
 </signals>
