File: EEprom_Logger_V1.sch (EAGLE design)
At the start: 18 parts, among them IC1 TC1016, IC2 PIC18F13K22SOP, IC3 MIC94090, IC4 24LCS21ASN, Q2 Si2333CDS-T1-GE3, Y1 32kHz

Commit message: Add files via upload
Parts:
- removed IC4: 24LCS21ASN, microchip:24LCS21ASN
- removed VBATT: Vbatt, SparkFun-Connectors:M02JST-PTH-2
- added IC5: 24LC16BSN, microchip:24LC16BSN
- added R2, R3: 4.7k, SparkFun-Resistors:RESISTOR1206
Connections:
- new net SCL: IC2.RB6/SCK, IC5.SCL, R2.1
- new net SDA: IC2.RB4/SDI, IC5.SDA, R3.1
- net GND: now also IC5.A0, IC5.A1, IC5.A2, IC5.GND, IC5.WP; no longer VBATT.2
- net SWITCHED_VCC: now also IC5.VCC, R2.2, R3.2
- net VIN: no longer VBATT.1
Other:
- note added: "18500 or AA LiFePO4 Battery 18500 needs 0.636'' spacer to fit into 18650 holder Use Super Cap (1F,2.7V + Boost Converter)"
- note removed: "18500 or AA LiFePO4 Battery 18500 needs 0.636'' spacer to fit into 18650 holder"
- note removed: "External Battery Connector"
